File: Balun/four-to-one-balun-v0.1/four-to-one-balun.kicad_pcb (KiCad board)
At the start: 2 copper layers, 69.8 x 71.1 mm, 8 parts, among them P1 N-TYPE, P2 N-TYPE, P3 N-TYPE, P4 CLAMP, P5 CLAMP

Commit message: Fix connector obstruction to antenna elements
Parts:
- moved P1 20.0 mm to (176.5, 121.0)
Routing:
- net GND: track 181.7 -> 268.9 mm, vias 5 -> 8
- net N-000003: track 66.6 -> 59.8 mm
Other:
- board text added: "4:1 Balun REV0.2 ©2015 Libre Space Foundation"
- board text removed: "4:1 Balun REV0.1 ©2015 Libre Space Foundation"
Changed lines of the file:
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@@
-(kicad_pcb (version 3) (host pcbnew "(25-Oct-2014 BZR 4029)-stable")
+(kicad_pcb (version 3) (host pcbnew "(22-Jun-2014 BZR 4027)-stable")
   (general
     (links 10)
@@
     (thickness 1.6)
     (drawings 5)
-    (tracks 29)
+    (tracks 34)
     (zones 0)
     (modules 8)
@@
   (title_block
     (title "4:1 Balun")
-    (rev 0.1)
+    (rev 0.2)
     (company "Libre Space Foundation")
   )
@@
   )
   (module NTYPE_EDGE (layer F.Cu)
-    (at 176.53 140.97 180)
+    (at 176.53 120.97 180)
     (fp_text reference P1 (at 10.16 -1.27 180) (layer F.SilkS)
       (effects (font (size 1.524 1.524) (thickness 0.3048)))
@@
     )
   )
-  (gr_text "4:1 Balun REV0.1\n©2015 Libre Space Foundation" (at 190.5 168.91) (layer F.Cu)
+  (gr_text "4:1 Balun REV0.2\n©2015 Libre Space Foundation" (at 190.5 168.91) (layer F.Cu)
     (effects (font (size 1.3 1.3) (thickness 0.3)) (justify left))
   )
@@
   (gr_line (start 176.53 105.41) (end 246.38 105.41) (angle 90) (layer Edge.Cuts) (width 0.1))
   (gr_line (start 176.53 176.53) (end 176.53 105.41) (angle 90) (layer Edge.Cuts) (width 0.1))
+  (segment (start 197.104 156.464) (end 211.836 156.464) (width 3) (layer B.Cu) (net 1))
+  (via (at 197.104 156.464) (size 2.54) (layers F.Cu B.Cu) (net 1))
+  (segment (start 181.61 140.97) (end 197.104 156.464) (width 3) (layer B.Cu) (net 1))
+  (via (at 217.932 150.368) (size 2.54) (layers F.Cu B.Cu) (net 1))
+  (segment (start 211.836 156.464) (end 217.932 150.368) (width 3) (layer B.Cu) (net 1))
+  (segment (start 181.61 140.97) (end 209.804 112.776) (width 3) (layer B.Cu) (net 1))
+  (via (at 211.836 112.776) (size 2.54) (layers F.Cu B.Cu) (net 1))
+  (segment (start 209.804 112.776) (end 211.836 112.776) (width 3) (layer B.Cu) (net 1))
+  (segment (start 196.85 140.97) (end 181.61 140.97) (width 3) (layer B.Cu) (net 1))
+  (segment (start 180.78 110.47) (end 180.78 113.47) (width 3) (layer F.Cu) (net 1))
+  (segment (start 180.78 113.47) (end 181.61 114.3) (width 3) (layer F.Cu) (net 1))
+  (via (at 181.61 114.3) (size 2.54) (layers F.Cu B.Cu) (net 1))
+  (segment (start 181.61 114.3) (end 181.61 140.97) (width 3) (layer B.Cu) (net 1))
+  (segment (start 181.61 132.3) (end 180.78 131.47) (width 3) (layer F.Cu) (net 1))
+  (via (at 181.61 140.97) (size 2.54) (layers F.Cu B.Cu) (net 1))
+  (segment (start 181.61 140.97) (end 181.61 132.3) (width 3) (layer F.Cu) (net 1))
   (segment (start 226.06 140.97) (end 241.3 140.97) (width 3) (layer B.Cu) (net 1))
   (segment (start 226.06 140.97) (end 196.85 140.97) (width 3) (layer B.Cu) (net 1))
-  (segment (start 196.85 140.97) (end 181.61 140.97) (width 3) (layer B.Cu) (net 1))
-  (segment (start 180.78 151.47) (end 180.78 155.38) (width 3) (layer F.Cu) (net 1))
-  (segment (start 180.78 126.56) (end 180.78 130.47) (width 3) (layer F.Cu) (net 1))
-  (segment (start 181.61 125.73) (end 180.78 126.56) (width 3) (layer F.Cu) (net 1))
-  (via (at 181.61 125.73) (size 2.54) (layers F.Cu B.Cu) (net 1))
-  (segment (start 181.61 156.21) (end 181.61 140.97) (width 3) (layer B.Cu) (net 1))
-  (segment (start 181.61 140.97) (end 181.61 125.73) (width 3) (layer B.Cu) (net 1))
-  (via (at 181.61 156.21) (size 2.54) (layers F.Cu B.Cu) (net 1))
-  (segment (start 180.78 155.38) (end 181.61 156.21) (width 3) (layer F.Cu) (net 1))
   (segment (start 241.3 140.97) (end 241.3 132.3) (width 3) (layer F.Cu) (net 1) (status 20))
   (segment (start 241.3 132.3) (end 242.13 131.47) (width 3) (layer F.Cu) (net 1) (status 30))
@@
   (segment (start 241.3 114.3) (end 242.13 113.47) (width 3) (layer F.Cu) (net 1))
   (via (at 241.3 114.3) (size 2.54) (layers F.Cu B.Cu) (net 1))
-  (segment (start 241.3 140.97) (end 241.3 114.3) (width 3) (layer B.Cu) (net 1) (status 2))
+  (segment (start 241.3 140.97) (end 241.3 114.3) (width 3) (layer B.Cu) (net 1))
   (segment (start 231.455 160.97) (end 240.63 160.97) (width 2.5) (layer F.Cu) (net 2))
+  (segment (start 180.78 120.97) (end 231.455 120.97) (width 2.5) (layer F.Cu) (net 3))
   (segment (start 240.63 120.97) (end 231.455 120.97) (width 2.5) (layer F.Cu) (net 3) (status 10))
-  (segment (start 182.28 140.97) (end 182.88 140.97) (width 2.5) (layer F.Cu) (net 3))
-  (segment (start 202.88 120.97) (end 231.455 120.97) (width 2.5) (layer F.Cu) (net 3))
-  (segment (start 182.88 140.97) (end 202.88 120.97) (width 2.5) (layer F.Cu) (net 3))
   (zone (net 1) (net_name GND) (layer B.Cu) (hatch edge 0.508)
     (connect_pads (clearance 0.508))
